File: 001_ESC/001_ESC.kicad_pcb (KiCad board)
At the start: 2 copper layers, 66 x 58.9 mm, 73 parts, among them IC1 MP2307DN-LF-Z, IC2 IR2101STRPBF, IC3 IR2101STRPBF, IC4 IR2101STRPBF, J1 USB_B_Micro, J2 Conn_01x05_Female, J3 Conn_01x03_Male, J4 Conn_01x03_Male, J5 Conn_01x02_Male, Q1 IRLR7843TRPBF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

Commit message: update.
Connections:
- J4 pad 1: PhaseB -> PhaseC
- Q5 pad 3: PhaseB -> PhaseC
- R20 pad 2: PhaseB -> PhaseC
Routing:
- net PhaseC: track 15.4 -> 72.5 mm, vias 0 -> 2
- net PhaseB: track 94.4 -> 71.6 mm
Other:
- board text added: "P.A"
- board text added: "P.B"
- board text added: "P.C"
- board text added: "PWM_INPUT"
- board text added: "UART_PINS"
- board text added: "VCC_GND"
