File: 001_ESC/001_ESC.kicad_sch (KiCad schematic)
At the start: 73 parts, among them IC1 MP2307DN-LF-Z, IC2 IR2101STRPBF, IC3 IR2101STRPBF, IC4 IR2101STRPBF, J1 USB_B_Micro, J2 Conn_01x05_Female, J3 Conn_01x03_Male, J4 Conn_01x03_Male, J5 Conn_01x02_Male, Q1 IRLR7843TRPBF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

Commit message: update.
Changed lines of the file:
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@@
     (stroke (width 0) (type default) (color 0 0 0 0))
   )
-  (wire (pts (xy 214.63 109.22) (xy 222.25 109.22))
+  (wire (pts (xy 214.63 109.22) (xy 215.9 109.22))
     (stroke (width 0) (type default) (color 0 0 0 0))
   )
@@
     (stroke (width 0) (type default) (color 0 0 0 0))
   )
-  (wire (pts (xy 129.54 99.06) (xy 129.54 95.25))
+  (wire (pts (xy 129.54 99.06) (xy 129.54 90.17))
     (stroke (width 0) (type default) (color 0 0 0 0))
   )
@@
     )
   )
-  (global_label "PhaseC" (shape input) (at 222.25 109.22 90) (fields_autoplaced)
+  (global_label "PhaseC" (shape input) (at 215.9 109.22 0) (fields_autoplaced)
     (effects (font (size 1 1)) (justify left))
-    (property "Intersheet References" "${INTERSHEET_REFS}" (id 0) (at 222.1875 101.8438 90)
+    (property "Intersheet References" "${INTERSHEET_REFS}" (id 0) (at 223.2762 109.1575 0)
       (effects (font (size 1 1)) (justify left) hide)
     )
@@
     )
   )
-  (global_label "PhaseB" (shape input) (at 129.54 95.25 90) (fields_autoplaced)
+  (global_label "PhaseB" (shape input) (at 129.54 90.17 0) (fields_autoplaced)
     (effects (font (size 1 1)) (justify left))
-    (property "Intersheet References" "${INTERSHEET_REFS}" (id 0) (at 129.4775 87.8738 90)
+    (property "Intersheet References" "${INTERSHEET_REFS}" (id 0) (at 136.9162 90.1075 0)
       (effects (font (size 1 1)) (justify left) hide)
     )
@@
   (symbol (lib_id "Connector:Conn_01x03_Male") (at 90.17 168.91 180) (unit 1)
     (in_bom yes) (on_board yes)
-    (property "Reference" "J4" (id 0) (at 89.535 176.53 0))
+    (property "Reference" "J4" (id 0) (at 90.17 172.72 0))
     (property "Value" "Conn_01x03_Male" (id 1) (at 92.71 168.91 90))
     (property "Footprint" "Connector_Wire:SolderWire-0.5sqmm_1x03_P4.8mm_D0.9mm_OD2.3mm" (id 2) (at 90.17 168.91 0)
